File: bussedBreakout0805.kicad_pcb (KiCad board)
At the start: 2 copper layers, 2.9 x 2.9 mm, 34 parts, among them J1 Conn_01x12_Pin, J10 Conn_01x06_Pin, J11 Conn_01x06_Pin, J12 Conn_01x06_Pin, J13 Conn_01x06_Pin, J14 Conn_01x06_Pin, J15 Conn_01x06_Pin, J16 Conn_01x06_Pin, J17 Conn_01x06_Pin, J18 Conn_01x06_Pin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

Commit message: Routing completed
Parts:
- added J21: Conn_01x06_Pin, SMD:SMD_0805_grid_1x6, F.Cu at (33.0, 27.9)
- added J22: Conn_01x06_Pin, SMD:SMD_0805_grid_1x6, F.Cu at (33.0, 30.5)
- added J23: Conn_01x06_Pin, SMD:SMD_0805_grid_1x6, F.Cu at (33.0, 33.0)
- added J24: Conn_01x06_Pin, SMD:SMD_0805_grid_1x6, F.Cu at (33.0, 35.6)
- added J25: Conn_01x06_Pin, SMD:SMD_0805_grid_1x6, F.Cu at (33.0, 38.1)
- added J26: Conn_01x06_Pin, SMD:SMD_0805_grid_1x6, F.Cu at (33.0, 40.6)
- added J27: Conn_01x06_Pin, SMD:SMD_0805_grid_1x6, F.Cu at (33.0, 43.2)
- added J28: Conn_01x06_Pin, SMD:SMD_0805_grid_1x6, F.Cu at (33.0, 45.7)
- added J29: Conn_01x06_Pin, SMD:SMD_0805_grid_1x6, F.Cu at (33.0, 48.3)
- added J30: Conn_01x06_Pin, SMD:SMD_0805_grid_1x6, F.Cu at (33.0, 50.8)
- added J31: Conn_01x06_Pin, SMD:SMD_0805_grid_1x6, F.Cu at (33.0, 53.3)
- added J32: Conn_01x06_Pin, SMD:SMD_0805_grid_1x6, F.Cu at (33.0, 55.9)
Routing:
- net /1: track 0.00 -> 6.72 mm, vias 0 -> 3
- net /9: track 0.00 -> 6.71 mm, vias 0 -> 3
- net /8: track 0.00 -> 6.71 mm, vias 0 -> 3
- net /7: track 0.00 -> 6.71 mm, vias 0 -> 3
- net /6: track 0.00 -> 6.71 mm, vias 0 -> 3
- net /5: track 0.00 -> 6.71 mm, vias 0 -> 3
- net /4: track 0.00 -> 6.71 mm, vias 0 -> 3
- net /3: track 0.00 -> 6.71 mm, vias 0 -> 3
- net /24: track 0.00 -> 6.71 mm, vias 0 -> 3
- net /23: track 0.00 -> 6.71 mm, vias 0 -> 3
- net /22: track 0.00 -> 6.71 mm, vias 0 -> 3
- net /21: track 0.00 -> 6.71 mm, vias 0 -> 3
- net /20: track 0.00 -> 6.71 mm, vias 0 -> 3
- net /2: track 0.00 -> 6.71 mm, vias 0 -> 3
- net /19: track 0.00 -> 6.71 mm, vias 0 -> 3
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Other:
- board text added: "1"
- board text added: "12"
- board text added: "13"
- board text added: "24"
- board text added: "A"
- board text added: "E"
