File: bussedBreakout0805.kicad_sch (KiCad schematic)
At the start: 34 parts, among them J1 Conn_01x12_Pin, J10 Conn_01x06_Pin, J11 Conn_01x06_Pin, J12 Conn_01x06_Pin, J13 Conn_01x06_Pin, J14 Conn_01x06_Pin, J15 Conn_01x06_Pin, J16 Conn_01x06_Pin, J17 Conn_01x06_Pin, J18 Conn_01x06_Pin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

Commit message: Routing completed
Parts:
- added J21, J22, J23, J24, J25, J26, J27, J28, J29, J30, J31, J32: Conn_01x06_Pin, SMD:SMD_0805_grid_1x6, symbol Connector:Conn_01x06_Pin
Connections:
- net 1: now also J21.1 (Pin_1), J21.2 (Pin_2), J21.3 (Pin_3)
- net 10: now also J30.1 (Pin_1), J30.2 (Pin_2), J30.3 (Pin_3)
- net 11: now also J31.1 (Pin_1), J31.2 (Pin_2), J31.3 (Pin_3)
- net 12: now also J32.1 (Pin_1), J32.2 (Pin_2), J32.3 (Pin_3)
- net 13: now also J32.4 (Pin_4), J32.5 (Pin_5), J32.6 (Pin_6)
- net 14: now also J31.4 (Pin_4), J31.5 (Pin_5), J31.6 (Pin_6)
- net 15: now also J30.4 (Pin_4), J30.5 (Pin_5), J30.6 (Pin_6)
- net 16: now also J29.4 (Pin_4), J29.5 (Pin_5), J29.6 (Pin_6)
- net 17: now also J28.4 (Pin_4), J28.5 (Pin_5), J28.6 (Pin_6)
- net 18: now also J27.4 (Pin_4), J27.5 (Pin_5), J27.6 (Pin_6)
- net 19: now also J26.4 (Pin_4), J26.5 (Pin_5), J26.6 (Pin_6)
- net 2: now also J22.1 (Pin_1), J22.2 (Pin_2), J22.3 (Pin_3)
- net 20: now also J25.4 (Pin_4), J25.5 (Pin_5), J25.6 (Pin_6)
- net 21: now also J24.4 (Pin_4), J24.5 (Pin_5), J24.6 (Pin_6)
- net 22: now also J23.4 (Pin_4), J23.5 (Pin_5), J23.6 (Pin_6)
- net 23: now also J22.4 (Pin_4), J22.5 (Pin_5), J22.6 (Pin_6)
- net 24: now also J21.4 (Pin_4), J21.5 (Pin_5), J21.6 (Pin_6)
- net 3: now also J23.1 (Pin_1), J23.2 (Pin_2), J23.3 (Pin_3)
- net 4: now also J24.1 (Pin_1), J24.2 (Pin_2), J24.3 (Pin_3)
- net 5: now also J25.1 (Pin_1), J25.2 (Pin_2), J25.3 (Pin_3)
- net 6: now also J26.1 (Pin_1), J26.2 (Pin_2), J26.3 (Pin_3)
- net 7: now also J27.1 (Pin_1), J27.2 (Pin_2), J27.3 (Pin_3)
- net 8: now also J28.1 (Pin_1), J28.2 (Pin_2), J28.3 (Pin_3)
- net 9: now also J29.1 (Pin_1), J29.2 (Pin_2), J29.3 (Pin_3)
Other:
- note added: "Breakout on top"
